File: hardware/Scorbot Driver/Scorbot Driver.kicad_sch (KiCad schematic)
At the start: 87 parts, among them Q1 2N7002, Q2 2N7002, Q3 2N7002, Q4 2N7002, Q5 2N7002, U1 24pin ATX PSU Connector, U10 OPB628, U11 OPB628, U2 Raspi Motor Driver HAT, U3 Raspi Motor Driver HAT, U4 MCP23017-E/SP, U5 ADS1015BQDGSRQ1, U6 MCP23017-E/SP, U7 ADS1015BQDGSRQ1, U8 ADS1015BQDGSRQ1, U9 ADS1015BQDGSRQ1

Commit message: schematics cleanup from migration
Parts:
- removed A: A, symbol Unknown_0_-1632
- R25, R26, R30, R31, R32, R33: value 1k -> 5k
Other:
- company: (none) -> Talos RIT
- title: (none) -> ScorBot Driver
- moved on the sheet: C1, Q1, Q2, Q3, Q4, Q5, R2, R37, R38, R39, R40, R41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

Commit message: esp32 added and logic level shifters added
Parts:
- removed Q2: 2N7002, symbol 2N7002_1
- removed Q3: 2N7002, symbol 2N7002_2
- removed Q4: 2N7002, symbol 2N7002_3
- removed Q5: 2N7002, symbol 2N7002_4
- removed R1: 0.1, symbol R_0603_US_1
- removed R12: 0.1, symbol R_0603_US_11
- removed R13: 10k, symbol R_0603_US_12
- removed R14: 10k, symbol R_0603_US_13
- removed R15: 5k, symbol R_0603_US_14
- removed R16: 5k, symbol R_0603_US_15
- removed R17: 5k, symbol R_0603_US_16
- removed R18: 5k, symbol R_0603_US_17
- removed R19: 10k, symbol R_0603_US_18
- removed R20: 10k, symbol R_0603_US_19
- removed R21: 0.1, symbol R_0603_US_20
- removed R22: 0.1, symbol R_0603_US_21
- removed R23: 10k, symbol R_0603_US_22
- removed R24: 10k, symbol R_0603_US_23
- removed R25: 5k, symbol R_0603_US_24
- removed R26: 5k, symbol R_0603_US_25
- removed R27: 0.1, symbol R_0603_US_26
- removed R28: 10k, symbol R_0603_US_27
- removed R29: 10k, symbol R_0603_US_28
- removed R3: 10k, symbol R_0603_US_2
- removed R30: 5k, symbol R_0603_US_29
- removed R31: 5k, symbol R_0603_US_30
- removed R32: 5k, symbol R_0603_US_31
- removed R33: 5k, symbol R_0603_US_32
- removed R34: 10k, symbol R_0603_US_33
- removed R35: 10k, symbol R_0603_US_34
- removed R36: 0.1, symbol R_0603_US_35
- removed R4: 10k, symbol R_0603_US_3
- removed R5: 5k, symbol R_0603_US_4
- removed R58: 1k, symbol R_0603_US_57
- removed R59: 1k, symbol R_0603_US_58
- removed R6: 5k, symbol R_0603_US_5
- removed R60: 1k, symbol R_0603_US_59
- removed R61: 1k, symbol R_0603_US_60
- removed R62: 1k, symbol R_0603_US_61
- removed R63: 1k, symbol R_0603_US_62
- removed R64: 1k, symbol R_0603_US_63
- removed R65: 1k, symbol R_0603_US_64
- removed U3: Raspi Motor Driver HAT, symbol Raspi Motor Driver HAT_1
- removed U4: MCP23017-E/SP, symbol MCP23017-E/SP_1
- removed U6: MCP23017-E/SP, symbol MCP23017-E/SP
- added C2, C? (x6): 100uF, symbol C_0603_US
- added D1, D10, D11, D12, D13, D14, D15, D16, D17, D18, D19, D2, D20, D21, D22, D23, D24, D25, D26, D29, D3, D30, D4, D5, D6, D7, D8, D9: SB550, Diode_THT:D_DO-201AD_P15.24mm_Horizontal, symbol Diode:1N5822
- added R1, R22, R31, R32, R6, R71: 5k, symbol R_0603_US_7
- added R12, R21, R23, R3, R30, R70: 15k, symbol R_0603_US_8
- added R15, R16, R17, R26, R27, R69: 0.1, symbol R_0603_US_10
- added R19, R25, R28, R33, R5, R67: 5k, symbol R_0603_US_6
- added R20, R24, R29, R34, R4, R66: 15k, symbol R_0603_US_9
- added R? (x7): 10, symbol R_0603_US_65
- added SW: SW_SPDT, symbol Switch:SW_SPDT
- added unit 1 of U1
- added U12: Raspi Motor Driver HAT, symbol Raspi Motor Driver HAT
- added U? (x4): Logic Level Shifter, symbol Converter_DCDC:LogicLevelShifter
- added U?: ESP32-S3-DevKitC, PCM_Espressif:ESP32-S3-DevKitC, symbol Espressif?:ESP32-S3-DevKitC
- R10, R9: value 10k -> 15k
- renumbered M to M1
Connections:
- net +5V: now also U1.6 (5V), R?.1, R?.1, R?.1, R?.1, R?.1, R?.1, R?.1, U1.9 (HV), U12.5 (5V), U?.21 (5V), U?.9 (HV), U?.9 (HV), U?.9 (HV), U?.9 (HV); no longer R51.2, R52.2, R53.2, R54.2, R55.2, U1.9 (5VSTBY)
- net 5VEncINTA: now also U1.7 (HV1)
- net 5VEncINTB: now also U1.8 (HV2)
- net 5VEncSCL: now also U1.12 (HV4)
- net 5VEncSDA: now also U1.11 (HV3)
- net Axis+: now also D23.2 (A), D24.1 (K), U12.12 (M3A)
- net Axis-: now also D19.2 (A), D20.1 (K), R17.1, R34.2
- net Axis1+: now also D7.2 (A), D8.1 (K)
- net Axis1-: now also D5.2 (A), D6.1 (K), R66.2, R69.1; no longer R10.2, R11.1
- net Axis1Limit: now also U?.20 (GPIO14/ADC2_CH3)
- net Axis1P0: now also U?.7 (HV1)
- net Axis1P1: now also U?.8 (HV2)
- net Axis1SENS1: now also R70.1, R71.2; no longer R10.1, R7.2
- net Axis1SENS2: no longer R8.2, R9.1
- net Axis1Vled: now also C?.1, R?.2
- net Axis2+: now also D1.2 (A), D4.1 (K)
- net Axis2-: now also R11.2, R9.2, D2.2 (A), D3.1 (K)
- net Axis2Limit: now also U?.10 (GPIO17/ADC2_CH6)
- net Axis2P0: now also U?.11 (HV3)
- net Axis2P1: now also U?.12 (HV4)
- net Axis2SENS1: now also R10.1, R7.2
- net Axis2SENS2: now also R8.2, R9.1
- net Axis2Vled: now also C?.1, R?.2
- net Axis3+: now also D11.2 (A), D12.1 (K)
- net Axis3-: now also D10.1 (K), D9.2 (A), R26.1, R29.2
- net Axis3Limit: now also U?.11 (GPIO18/ADC2_CH7)
- net Axis3P0: now also U?.7 (HV1)
- net Axis3P1: now also U?.8 (HV2)
- net Axis3SENS1: now also R22.2, R23.1
- net Axis3Vled: now also C?.1, R?.2
- net Axis4+: now also D13.2 (A), D14.1 (K)
- net Axis4-: now also D15.2 (A), D16.1 (K), R27.2, R30.2
- net Axis4Limit: now also U?.27 (GPIO21)
- net Axis4P0: now also U?.11 (HV3)
- net Axis4P1: now also U?.12 (HV4)
- net Axis4SENS1: now also R24.1, R25.2
- net Axis4SENS2: now also R30.1, R31.2
- net Axis4Vled: now also C?.1, R?.2
- net Axis5+: now also D21.2 (A), D22.1 (K), U12.7 (M1A)
- net Axis5-: now also D17.2 (A), D18.1 (K), R15.1, R20.2
- net Axis5Limit: now also U?.32 (GPIO35)
- net Axis5P0: now also U?.7 (HV1)
- net Axis5P1: now also U?.8 (HV2)
- net Axis5SENS1: now also R1.2, R3.1
- net Axis5Vled: now also C?.1, R?.2
- net AxisP0: now also U?.7 (HV1)
- net AxisP1: now also U?.8 (HV2)
- net AxisSENS1: now also R12.1, R6.2
- net AxisVled: now also C2.1, R?.2
- net GND: now also C2.2, C?.2, C?.2, C?.2, C?.2, C?.2, C?.2, D10.2 (A), D12.2 (A), D14.2 (A), D16.2 (A), D18.2 (A), D20.2 (A), D22.2 (A), D24.2 (A), D26.2 (A), D3.2 (A), D30.2 (A), D4.2 (A), D6.2 (A), D8.2 (A), R1.1, R19.1, R22.1, R25.1, R28.1, R31.1, R32.1, R33.1, R5.1, R6.1, R67.1, R71.1, U1.10 (GND), U1.4 (GND), U12.6 (GND), U?.10 (GND), U?.10 (GND), U?.10 (GND), U?.10 (GND), U?.22 (GND), U?.23 (GND), U?.24 (GND), U?.4 (GND), U?.4 (GND), U?.4 (GND), U?.4 (GND), U?.44 (GND)
- net Gripper+: now also D25.2 (A), D26.1 (K), U12.10 (M2A)
- net Gripper-: now also D29.2 (A), D30.1 (K), R16.2, R21.2
- net GripperP0: now also U?.11 (HV3)
- net GripperP1: now also U?.12 (HV4)
- net GripperSENS1: now also R4.1, R5.2
- net GripperSENS2: now also R21.1, R32.2
- net GripperVled: now also C?.1, R?.2
- net MotSCL: now also U12.1 (SCL)
- net MotSDA: now also U12.2 (SDA)
- net VCC: now also R51.2, R52.2, R53.2, R54.2, R55.2, U1.3 (LV), U12.4 (3.3V), U?.1 (3V3), U?.2 (3V3), U?.3 (LV), U?.3 (LV), U?.3 (LV), U?.3 (LV)
- net VCCEncINTA: now also U1.1 (LV1)
- net VCCEncINTB: now also U1.2 (LV2)
- net VCCEncSCL: now also U1.6 (LV4)
- net VCCEncSDA: now also U1.5 (LV3)
- net at M1.16 (GPIO23): now also U5.2 (ALERT/RDY)
- net at M1.18 (GPIO24): now also U7.2 (ALERT/RDY)
- net at M1.22 (GPIO25): now also U8.2 (ALERT/RDY)
- net at M1.24 (GPIO8): now also U9.2 (ALERT/RDY)
- net at U1.19 (GND): now also SW.3 (C)
- removed net Axis1FromMotor: R11.2, R9.2, U2.9 (M1B)
- net Axis2FromMotor: no longer names the net of U2.11 (M2B)
- net Axis2FromMotor: now also R10.2, R11.1
- net Axis3FromMotor: no longer names the net of U2.13 (M3B)
- net Axis3FromMotor: now also R23.2, R26.2
- net Axis4FromMotor: no longer names the net of U2.15 (M4B)
- net Axis4FromMotor: now also R24.2, R27.1
- net PS_On: no longer names the net of U1.16 (PS_ON)
- net PS_On: now also SW.2 (B)
- net PW_Good: no longer names the net of U1.8 (PW_G)
- net Vmotor renamed +12V
- net +12V: now also D1.1 (K), D11.1 (K), D13.1 (K), D15.1 (K), D17.1 (K), D19.1 (K), D2.1 (K), D21.1 (K), D23.1 (K), D25.1 (K), D29.1 (K), D5.1 (K), D7.1 (K), D9.1 (K), U12.3 (VMotor)
- new net: R12.2, R17.2, U12.13 (M3B)
- new net: R69.2, R70.2, U2.9 (M1B)
- new net: U?.1 (LV1), U?.31 (GPIO0)
- new net: U?.2 (LV2), U?.41 (GPIO1/ADC1_CH0)
- new net: U?.40 (GPIO2/ADC1_CH1), U?.5 (LV3)
- new net: U?.13 (GPIO3/ADC1_CH2), U?.6 (LV4)
- new net: R19.2, R20.1
- new net: U?.1 (LV1), U?.18 (GPIO12/ADC2_CH1)
- new net: U?.19 (GPIO13/ADC2_CH2), U?.2 (LV2)
- new net: R33.2, R34.1
- new net: R66.1, R67.2
- new net: R28.2, R29.1
- new net: R15.2, R3.2, U12.9 (M1B)
- new net: R16.1, R4.2, U12.11 (M2B)
- new net: U?.1 (LV1), U?.12 (GPIO8/ADC1_CH7)
- new net: U?.15 (GPIO9/ADC1_CH8), U?.2 (LV2)
- new net: U?.16 (GPIO10/ADC1_CH9), U?.5 (LV3)
- new net: U?.17 (GPIO11/ADC2_CH0), U?.6 (LV4)
- new net: U?.1 (LV1), U?.4 (GPIO4/ADC1_CH3)
- new net: U?.2 (LV2), U?.5 (GPIO5/ADC1_CH4)
- new net: U?.5 (LV3), U?.6 (GPIO6/ADC1_CH5)
- new net: U?.6 (LV4), U?.7 (GPIO7/ADC1_CH6)
- no-connect marks 37 -> 34
Other:
- note added: "+ to A, - to B"
- note added: "Emergency-stop"
- note added: "Inductive Kickback Protection"
- note added: "RC circuit to limit current to encoder diodes"
- note added: "This circuit is unchangeable!"
- note added: "Voltage Divider to convert 12v to ~3 volt"
- note removed: "RC circuit to limit current to diodes"
- note removed: "Voltage Divider to convert 12v to ~5 volt"
- moved on the sheet: C1, DB1, M1, Q1, R10, R11, R2, R56, R57, R68, R7, R8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

Commit message: esp32 hookup with paralleled limit switches
Parts:
- removed M1: RasiPi4B, symbol RasiPi4B
- removed Q1: 2N7002, symbol 2N7002
- removed R51: 1k, symbol R_0603_US_50
- removed R52: 1k, symbol R_0603_US_51
- removed R54: 1k, symbol R_0603_US_53
- removed R55: 1k, symbol R_0603_US_54
- removed R56: 1k, symbol R_0603_US_55
- removed R57: 1k, symbol R_0603_US_56
- removed unit 1 of U1
- removed U? (x4): Logic Level Shifter, symbol Converter_DCDC:LogicLevelShifter
- removed U?: ESP32-S3-DevKitC, PCM_Espressif:ESP32-S3-DevKitC, symbol Espressif?:ESP32-S3-DevKitC
- added R13, R14, R18: 1k, symbol R_0603_US_46
- added R35: 10k, symbol R_0603_US_46
- added U3: ESP32-DevKitC, PCM_Espressif:ESP32-DevKitC, symbol Espressif?:ESP32-DevKitC
- C1, C2: value 100uF -> 0.1uF
- R37, R38, R39, R40, R41, R42, R43, R44, R45, R46, R47, R48, R49, R50: value 1k -> 10k
- R68, R?: value 10 -> 47
Connections:
- net Axis2Limit is gone; now on net Axis1Limit: DSUB1.7
- net Axis3Limit is gone; now on net Axis1Limit: DSUB1.24, R53.1
- net Axis4Limit is gone; now on net Axis1Limit: DSUB1.8
- net Axis5Limit is gone; now on net Axis1Limit: DSUB1.6
- net +5V: now also U3.19 (5V); no longer R37.2, R38.2, R39.2, R40.2, R41.2, R42.2, R43.2, R44.2, R45.2, R46.2, R47.2, R48.2, R49.2, R50.2
- net Axis1P0: now also U3.3 (SENSOR_VP/GPIO36/ADC1_CH0)
- net Axis1P1: now also U3.4 (SENSOR_VN/GPIO39/ADC1_CH3)
- net Axis2P0: now also U3.5 (VDET_1/GPIO34/ADC1_CH6)
- net Axis2P1: now also U3.6 (VDET_2/GPIO35/ADC1_CH7)
- net Axis3P0: now also U3.7 (32K_XP/GPIO32/ADC1_CH4)
- net Axis3P1: now also U3.8 (32K_XN/GPIO33/ADC1_CH5)
- net Axis4P0: now also U3.9 (DAC_1/ADC2_CH8/GPIO25)
- net Axis4P1: now also U3.10 (DAC_2/ADC2_CH9/GPIO26)
- net Axis5P0: now also U3.11 (ADC2_CH7/GPIO27)
- net Axis5P1: now also U3.12 (MTMS/GPIO14/ADC2_CH6)
- net AxisP0: now also U3.27 (GPIO16)
- net AxisP1: now also U3.28 (GPIO17)
- net GND: now also U3.14 (GND), U3.32 (GND), U3.38 (GND)
- net GripperP0: now also U3.15 (MTCK/GPIO13/ADC2_CH4)
- net GripperP1: now also U3.26 (ADC2_CH0/GPIO4)
- net MotSCL: now also U3.36 (GPIO22)
- net MotSDA: now also U3.33 (GPIO21)
- net VCC: now also R37.2, R38.2, R39.2, R40.2, R41.2, R42.2, R43.2, R44.2, R45.2, R46.2, R47.2, R48.2, R49.2, R50.2, R13.2, R14.2, R18.2, R35.2
- net 1/2 ALRT: now reaches U5.2 (ALERT/RDY)
- net 1/2 ALRT: now also R13.1, U3.30 (GPIO18)
- net 3/4 ALRT: now reaches U7.2 (ALERT/RDY)
- net 3/4 ALRT: now also R14.1, U3.31 (GPIO19)
- net 5/GR ALRT: now reaches U8.2 (ALERT/RDY)
- net 5/GR ALRT: now also R18.1, U3.34 (U0RXD/GPIO3)
- net AUX ALRT: now reaches U9.2 (ALERT/RDY)
- net AUX ALRT: now also R35.1, U3.35 (U0TXD/GPIO1)
- new net Limit: U3.37 (GPIO23)
- no-connect marks 34 -> 43
Other:
- note added: "GPIO 4 'technically' isn't a strapping pin on the ESP32, but it IS on the ESP32-S3."
- note added: "GPIO 6-11 reserved for SPI Flash (flash mem to RAM) GPIO 0,2,4,12,15 reserved for bootloader (strapping pins)"
- note added: "Limit Switch Pull-up Resistor(s)"
- note added: "Pull up for alert pins If using Adafruit breakout board, a 10k pullup is onboard so these are not needed"
- note added: "Resistor divider should divide by 4, 10K+3.3K is fine too"
- note removed: "(Breakout Board)"
- note removed: "3.3V to 5V bi-di"
- note removed: "Limit Switch Pull-up Resistors"
- note removed: "Logic Level Shifter"
- moved on the sheet: R38, R39, R40, R41, R42, R43, R44, R45, R46, R47, R48, R49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
