File: hardware/Scorbot Driver/Scorbot Driver.kicad_sch (KiCad schematic)
At the start: 112 parts, among them U1 24pin ATX PSU Connector, U10 OPB628, U11 OPB628, U12 Raspi Motor Driver HAT, U2 Raspi Motor Driver HAT, U3 ESP32-DevKitC, U5 ADS1015BQDGSRQ1, U7 ADS1015BQDGSRQ1, U8 ADS1015BQDGSRQ1, U9 ADS1015BQDGSRQ1

Commit message: schematic update
Parts:
- added D15: SB550, Diode_THT:D_DO-201AD_P15.24mm_Horizontal, symbol Diode:1N5822
Connections:
- net +12V: now also D15.1 (K)
- net Axis4-: now also D15.2 (A)
- no-connect marks 44 -> 43
Changed lines of the file:
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@@
 	)
 	(no_connect
-		(at 422.91 340.36)
-	)
-	(no_connect
 		(at 521.97 281.94)
 	)
@@
 		)
 	)
-	(wire
-		(pts
-			(xy 491.49 93.98) (xy 483.87 93.98)
-		)
-		(stroke
-			(width 0)
-			(type default)
-		)
-	)
-	(wire
-		(pts
-			(xy 397.51 101.6) (xy 387.35 101.6)
-		)
-		(stroke
-			(width 0)
-			(type default)
-		)
-	)
-	(wire
-		(pts
-			(xy 408.94 121.92) (xy 402.59 121.92)
-		)
-		(stroke
-			(width 0)
-			(type default)
-		)
-	)
-	(wire
-		(pts
-			(xy 416.56 106.68) (xy 416.56 104.14)
-		)
-		(stroke
-			(width 0)
-			(type default)
-		)
-	)
-	(wire
-		(pts
-			(xy 226.06 114.3) (xy 262.89 114.3)
-		)
-		(stroke
-			(width 0)
-			(type default)
-		)
-	)
-	(wire
-		(pts
-			(xy 520.7 82.55) (xy 530.86 82.55)
-		)
-		(stroke
-			(width 0)
-			(type default)
-		)
-	)
-	(wire
-		(pts
-			(xy 546.1 36.83) (xy 546.1 38.1)
-		)
-		(stroke
-			(width 0)
-			(type default)
-		)
-	)
-	(wire
-		(pts
-			(xy 49.53 341.63) (xy 54.61 341.63)
-		)
-		(stroke
-			(width 0)
-			(type default)
-		)
-	)
-	(wire
-		(pts
-			(xy 416.56 52.07) (xy 430.53 52.07)
-		)
-		(stroke
-			(width 0)
-			(type default)
-		)
-	)
-	(wire
-		(pts
-			(xy 226.06 67.31) (xy 262.89 67.31)
-		)
-		(stroke
-			(width 0)
-			(type default)
-		)
-	)
-	(wire
-		(pts
-			(xy 539.75 115.57) (xy 539.75 121.92)
-		)
-		(stroke
-			(width 0)
-			(type default)
-		)
-	)
-	(wire
-		(pts
-			(xy 547.37 59.69) (xy 553.72 59.69)
-		)
-		(stroke
-			(width 0)
-			(type default)
-		)
-	)
-	(wire
-		(pts
-			(xy 494.03 88.9) (xy 483.87 88.9)
-		)
-		(stroke
-			(width 0)
-			(type default)
-		)
-	)
-	(wire
-		(pts
-			(xy 407.67 31.75) (xy 396.24 31.75)
-		)
-		(stroke
-			(width 0)
-			(type default)
-		)
-	)
 	(polyline
 		(pts
@@
 		)
 	)
-	(wire
-		(pts
-			(xy 419.1 39.37) (xy 419.1 36.83)
-		)
-		(stroke
-			(width 0)
-			(type default)
-		)
-	)
 	(polyline
 		(pts
@@
 		)
 	)
-	(wire
-		(pts
-			(xy 193.04 77.47) (xy 223.52 77.47)
-		)
-		(stroke
-			(width 0)
-			(type default)
-		)
-	)
-	(wire
-		(pts
-			(xy 542.29 54.61) (xy 485.14 54.61)
-		)
-		(stroke
-			(width 0)
-			(type default)
-		)
-	)
 	(global_label "Axis3+"
 		(shape input)
@@
 	(global_label "Axis1P1"
 		(shape input)
-		(at 285.75 105.41 180)
+		(at 285.75 105.41 0)
 		(effects
 			(font
@@
 			)
 		)
-		(pin "2"
-		)
 		(pin "1"
